File: ghostlight/mcu.kicad_sch (KiCad schematic)
At the start: 4 parts, among them IC1 STM32C011J4M6

Commit message: change in schematic
Connections:
- net LIVE: now reaches IC1.5 (PA11[PA9]/PA8)
- net I2C_ERR: now reaches IC1.6 (PA12[PA10])
- no-connect marks 2 -> 0
Changed lines of the file:
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@@
-	)
-	(junction
-		(at 158.75 63.5)
-		(diameter 0)
-		(color 0 0 0 0)
 	)
 	(junction
@@
 	)
 	(junction
+		(at 166.37 63.5)
+		(diameter 0)
+		(color 0 0 0 0)
+	)
+	(junction
 		(at 171.45 34.29)
 		(diameter 0)
@@
 		(color 0 0 0 0)
 	)
-	(no_connect
-		(at 146.05 71.12)
-	)
-	(no_connect
-		(at 146.05 68.58)
-	)
 	(wire
 		(pts
@@
 	(wire
 		(pts
-			(xy 158.75 63.5) (xy 158.75 137.16)
+			(xy 166.37 63.5) (xy 166.37 68.58)
 		)
 		(stroke
@@
 	(wire
 		(pts
-			(xy 146.05 63.5) (xy 158.75 63.5)
+			(xy 146.05 63.5) (xy 166.37 63.5)
+		)
+		(stroke
+			(width 0)
+			(type default)
+		)
+	)
+	(wire
+		(pts
+			(xy 152.4 68.58) (xy 146.05 68.58)
 		)
 		(stroke
@@
 	(wire
 		(pts
-			(xy 119.38 137.16) (xy 119.38 165.1)
+			(xy 247.65 68.58) (xy 247.65 146.05)
 		)
 		(stroke
@@
 	(wire
 		(pts
-			(xy 158.75 137.16) (xy 119.38 137.16)
+			(xy 247.65 68.58) (xy 166.37 68.58)
 		)
 		(stroke
@@
 	(wire
 		(pts
-			(xy 151.13 66.04) (xy 151.13 130.81)
+			(xy 162.56 66.04) (xy 162.56 72.39)
 		)
 		(stroke
@@
 	(wire
 		(pts
+			(xy 166.37 63.5) (xy 171.45 63.5)
+		)
+		(stroke
+			(width 0)
+			(type default)
+		)
+	)
+	(wire
+		(pts
 			(xy 64.77 34.29) (xy 64.77 63.5)
 		)
@@
 	(wire
 		(pts
-			(xy 151.13 130.81) (xy 109.22 130.81)
+			(xy 237.49 72.39) (xy 162.56 72.39)
 		)
 		(stroke
@@
 	(wire
 		(pts
-			(xy 146.05 66.04) (xy 151.13 66.04)
+			(xy 146.05 66.04) (xy 162.56 66.04)
 		)
 		(stroke
@@
 	(wire
 		(pts
-			(xy 158.75 63.5) (xy 171.45 63.5)
-		)
-		(stroke
-			(width 0)
-			(type default)
-		)
-	)
-	(wire
-		(pts
 			(xy 171.45 57.15) (xy 171.45 63.5)
 		)
@@
 	(wire
 		(pts
-			(xy 109.22 130.81) (xy 109.22 165.1)
+			(xy 237.49 72.39) (xy 237.49 146.05)
 		)
 		(stroke
@@
 	(wire
 		(pts
+			(xy 146.05 142.24) (xy 146.05 71.12)
+		)
+		(stroke
+			(width 0)
+			(type default)
+		)
+	)
+	(wire
+		(pts
 			(xy 41.91 52.07) (xy 41.91 55.88)
 		)
@@
 		)
 	)
+	(wire
+		(pts
+			(xy 152.4 142.24) (xy 152.4 68.58)
+		)
+		(stroke
+			(width 0)
+			(type default)
+		)
+	)
 	(global_label "ST_LINK_SWDIO"
 		(shape input)
-		(at 109.22 165.1 270)
-		(fields_autoplaced yes)
-		(effects
-			(font
-				(size 1.27 1.27)
-			)
-			(justify right)
-		)
-		(property "Intersheetrefs" "${INTERSHEET_REFS}"
-			(at 109.22 182.2971 90)
+		(at 237.49 146.05 270)
+		(fields_autoplaced yes)
+		(effects
+			(font
+				(size 1.27 1.27)
+			)
+			(justify right)
+		)
+		(property "Intersheetrefs" "${INTERSHEET_REFS}"
+			(at 237.49 163.2471 90)
 			(hide yes)
 			(show_name no)
@@
 		)
 	)
+	(global_label "I2C_ERR"
+		(shape input)
+		(at 152.4 142.24 270)
+		(fields_autoplaced yes)
+		(effects
+			(font
+				(size 1.27 1.27)
+			)
+			(justify right)
+		)
+		(property "Intersheetrefs" "${INTERSHEET_REFS}"
+			(at 152.4 152.9661 90)
+			(hide yes)
+			(show_name no)
+			(do_not_autoplace no)
+			(effects
+				(font
+					(size 1.27 1.27)
+				)
+				(justify right)
+			)
+		)
+	)
 	(global_label "ST_LINK_RST{slash}RST"
 		(shape input)
@@
 		)
 	)
+	(global_label "LIVE"
+		(shape input)
+		(at 146.05 142.24 270)
+		(effects
+			(font
+				(size 1.27 1.27)
+			)
+			(justify right)
+		)
+		(property "Intersheetrefs" "${INTERSHEET_REFS}"
+			(at 146.05 142.24 90)
+			(hide yes)
+			(show_name no)
+			(do_not_autoplace no)
+			(effects
+				(font
+					(size 1.27 1.27)
+				)
+			)
+		)
+	)
 	(global_label "ST_LIKN_SWCLK"
 		(shape input)
-		(at 119.38 165.1 270)
-		(fields_autoplaced yes)
-		(effects
-			(font
-				(size 1.27 1.27)
-			)
-			(justify right)
-		)
-		(property "Intersheetrefs" "${INTERSHEET_REFS}"
-			(at 119.38 182.6599 90)
-			(hide yes)
-			(show_name no)
+		(at 247.65 146.05 270)
+		(fields_autoplaced yes)
+		(effects
+			(font
+				(size 1.27 1.27)
+			)
+			(justify right)
+		)
+		(property "Intersheetrefs" "${INTERSHEET_REFS}"
+			(at 247.65 163.6099 90)
+			(hide yes)
+			(show_name no)
