File: ghostlight/led.kicad_sch (KiCad schematic)
At the start: 3 parts, among them IC3 LP5817DRLR

Commit message: Add Test Points
Parts:
- added BLUE1: TP_B, TestPoint:TestPoint_Pad_D1.0mm, symbol Connector:TestPoint
- added GREEN1: TP_G, TestPoint:TestPoint_Pad_D1.0mm, symbol Connector:TestPoint
- added RED1: TP_R, TestPoint:TestPoint_Pad_D1.0mm, symbol Connector:TestPoint
Connections:
- net at IC3.6 (OUT2), LED1.3 (K_B): now also BLUE1.1
- net at IC3.7 (OUT1), LED1.2 (K_G): now also GREEN1.1
- net at IC3.8 (OUT0), LED1.1 (K_R): now also RED1.1
