File: ghostlight_circuit/ghostlight.kicad_pcb (KiCad board)
At the start: 2 copper layers, 27 x 27 mm, 15 parts, among them IC1 STM32C011J4M6, IC2 MCP1700T-3302E_TT, IC3 LP5817DRLR, J1 Conn_01x08

Commit message: rerouted the board
Parts:
- moved GREEN1 11.5 mm to (153.5, 96.5)
- moved RED1 11.5 mm to (155.5, 96.5)
- moved BLUE1 11.0 mm to (151.5, 96.5)
- moved C4 4.74 mm to (149.0, 94.5), turned to 0 degrees
- moved IC2 2.95 mm to (148.0, 101.0), turned to 180 degrees
- moved R2 2.31 mm to (155.5, 93.2), turned to -90 degrees
- moved IC3 2.30 mm to (152.0, 93.0), turned to 0 degrees
- moved C1 1.58 mm to (149.5, 105.0), turned to 90 degrees
- moved R1 1.53 mm to (157.0, 93.2), turned to -90 degrees
- moved C2 1.50 mm to (147.8, 97.5)
- moved C3 1.12 mm to (160.0, 95.0), turned to 180 degrees
- moved IC1 0.80 mm to (160.0, 99.5)
- renumbered BLUE to BLUE1, GREEN to GREEN1, RED to RED1
Connections:
- IC1 pad 5: LIVE -> SCK
- IC1 pad 8: SCK -> ST_LIKN_SWCLK
- J1 pad 2: SCK -> ST_LIKN_SWCLK
- J1 pad 5: LIVE -> unconnected-(J1-Pin_5-Pad5)
- J1 pad 7: unconnected-(J1-Pin_7-Pad7) -> V_BAT
Routing:
- net V_BAT: track 44.4 -> 16.8 mm, vias 3 -> 1
- net LIVE: track 12.5 -> 0.00 mm
- net ST_LIKN_SWCLK: track 0.00 -> 10.6 mm
- net Net-(IC3-OUT2): track 23.3 -> 15.4 mm, vias 0 -> 2
- net Net-(IC3-OUT0): track 16.4 -> 8.91 mm
- net SCK: track 23.0 -> 16.6 mm
- net ST_LINK_RST/RST: track 25.5 -> 19.6 mm
- net Net-(IC3-OUT1): track 15.7 -> 10.0 mm, vias 2 -> 0
- net GND: track 13.3 -> 11.8 mm
- net SDA: track 16.2 -> 17.6 mm
- net ST_LINK_SWDIO: track 8.16 -> 6.96 mm
- net I2C_ERR: track 5.85 -> 6.59 mm
Other:
- board size 27 x 27 mm -> 27 x 27.5 mm
