File: ghostlight_circuit/ghostlight.kicad_pcb (KiCad board)
At the start: 2 copper layers, 27 x 27.5 mm, 15 parts, among them IC1 STM32C011J4M6, IC2 MCP1700T-3302E_TT, IC3 LP5817DRLR, J1 Conn_01x08

Commit message: rebase scheme repair
Connections:
- J1 pad 6: ST_LINK_RST/RST -> unconnected-(J1-Pin_6-Pad6)
Routing:
- net 3.3V: track 63.6 -> 66.2 mm
- net Net-(IC3-OUT2): track 11.8 -> 10.2 mm

Commit message: TMP: added output files
Other:
- board size 27 x 27.5 mm -> 27 x 27 mm
