File: ghostlight_circuit/mcu.kicad_sch (KiCad schematic)
At the start: 4 parts, among them IC1 STM32C011J4M6

Commit message: rerouted the board
Connections:
- net LIVE is gone; now on net SCK: IC1.5 (PA11[PA9]/PA8)
- net SCK: no longer IC1.8 (PB6/PA14-BOOT0/PC15-OSCX_OUT)
- new net ST_LIKN_SWCLK: IC1.8 (PB6/PA14-BOOT0/PC15-OSCX_OUT)
Changed lines of the file:
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@@
 	(paper "A4")
 	(junction
+		(at 54.61 46.99)
+		(diameter 0)
+		(color 0 0 0 0)
+	)
+	(junction
+		(at 59.69 66.04)
+		(diameter 0)
+		(color 0 0 0 0)
+	)
+	(junction
 		(at 171.45 63.5)
 		(diameter 0)
@@
 	)
 	(junction
-		(at 54.61 46.99)
-		(diameter 0)
-		(color 0 0 0 0)
-	)
-	(junction
-		(at 59.69 66.04)
-		(diameter 0)
-		(color 0 0 0 0)
-	)
-	(junction
 		(at 54.61 57.15)
 		(diameter 0)
@@
 	)
 	(junction
-		(at 166.37 63.5)
-		(diameter 0)
-		(color 0 0 0 0)
-	)
-	(junction
 		(at 171.45 34.29)
 		(diameter 0)
@@
 	(wire
 		(pts
-			(xy 166.37 63.5) (xy 171.45 63.5)
-		)
-		(stroke
-			(width 0)
-			(type default)
-		)
-	)
-	(wire
-		(pts
 			(xy 64.77 34.29) (xy 64.77 63.5)
 		)
@@
 	(wire
 		(pts
+			(xy 146.05 71.12) (xy 171.45 71.12)
+		)
+		(stroke
+			(width 0)
+			(type default)
+		)
+	)
+	(wire
+		(pts
 			(xy 146.05 66.04) (xy 162.56 66.04)
 		)
@@
 	(wire
 		(pts
+			(xy 171.45 63.5) (xy 171.45 71.12)
+		)
+		(stroke
+			(width 0)
+			(type default)
+		)
+	)
+	(wire
+		(pts
 			(xy 67.31 71.12) (xy 67.31 165.1)
 		)
@@
 	(wire
 		(pts
-			(xy 146.05 142.24) (xy 146.05 71.12)
-		)
-		(stroke
-			(width 0)
-			(type default)
-		)
-	)
-	(wire
-		(pts
 			(xy 41.91 52.07) (xy 41.91 55.88)
 		)
@@
 			)
 		)
-	)
-	(global_label "LIVE"
-		(shape input)
-		(at 146.05 142.24 270)
-		(effects
-			(font
-				(size 1.27 1.27)
-			)
-			(justify right)
-		)
-		(property "Intersheetrefs" "${INTERSHEET_REFS}"
-			(at 146.05 142.24 90)
-			(hide yes)
-			(show_name no)
-			(do_not_autoplace no)
-			(effects
-				(font
-					(size 1.27 1.27)
-				)
-			)
-		)
