File: ghostlight_circuit/mcu.kicad_sch (KiCad schematic)
At the start: 4 parts, among them IC1 STM32C011J4M6

Commit message: update pcb
rerout and connect accelerometer

better re-route
Connections:
- net LIVE is gone; now on net SCK: IC1.5 (PA11[PA9]/PA8)
- net SCK: no longer IC1.8 (PB6/PA14-BOOT0/PC15-OSCX_OUT)
- net I2C_ERR renamed ACC_INT1
- new net ST_LIKN_SWCLK: IC1.8 (PB6/PA14-BOOT0/PC15-OSCX_OUT)
Changed lines of the file:
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@@
-	)
-	(junction
-		(at 166.37 63.5)
-		(diameter 0)
-		(color 0 0 0 0)
 	)
 	(junction
@@
 	(wire
 		(pts
-			(xy 166.37 63.5) (xy 166.37 68.58)
+			(xy 166.37 63.5) (xy 166.37 71.12)
 		)
 		(stroke
@@
 	(wire
 		(pts
-			(xy 146.05 63.5) (xy 166.37 63.5)
-		)
-		(stroke
-			(width 0)
-			(type default)
-		)
-	)
-	(wire
-		(pts
-			(xy 152.4 68.58) (xy 146.05 68.58)
+			(xy 175.26 142.24) (xy 175.26 147.32)
 		)
 		(stroke
@@
 	(wire
 		(pts
-			(xy 247.65 68.58) (xy 247.65 146.05)
-		)
-		(stroke
-			(width 0)
-			(type default)
-		)
-	)
-	(wire
-		(pts
 			(xy 25.4 39.37) (xy 54.61 39.37)
 		)
@@
 	(wire
 		(pts
-			(xy 247.65 68.58) (xy 166.37 68.58)
-		)
-		(stroke
-			(width 0)
-			(type default)
-		)
-	)
-	(wire
-		(pts
 			(xy 59.69 66.04) (xy 59.69 165.1)
 		)
@@
 	(wire
 		(pts
+			(xy 156.21 142.24) (xy 175.26 142.24)
+		)
+		(stroke
+			(width 0)
+			(type default)
+		)
+	)
+	(wire
+		(pts
 			(xy 54.61 66.04) (xy 59.69 66.04)
 		)
@@
 	(wire
 		(pts
+			(xy 146.05 63.5) (xy 156.21 63.5)
+		)
+		(stroke
+			(width 0)
+			(type default)
+		)
+	)
+	(wire
+		(pts
+			(xy 166.37 71.12) (xy 146.05 71.12)
+		)
+		(stroke
+			(width 0)
+			(type default)
+		)
+	)
+	(wire
+		(pts
+			(xy 153.67 148.59) (xy 153.67 68.58)
+		)
+		(stroke
+			(width 0)
+			(type default)
+		)
+	)
+	(wire
+		(pts
 			(xy 171.45 57.15) (xy 171.45 63.5)
 		)
@@
 	(wire
 		(pts
+			(xy 153.67 68.58) (xy 146.05 68.58)
+		)
+		(stroke
+			(width 0)
+			(type default)
+		)
+	)
+	(wire
+		(pts
 			(xy 48.26 55.88) (xy 48.26 68.58)
 		)
@@
 	(wire
 		(pts
-			(xy 146.05 142.24) (xy 146.05 71.12)
-		)
-		(stroke
-			(width 0)
-			(type default)
-		)
-	)
-	(wire
-		(pts
 			(xy 41.91 52.07) (xy 41.91 55.88)
 		)
@@
 	(wire
 		(pts
+			(xy 156.21 63.5) (xy 156.21 142.24)
+		)
+		(stroke
+			(width 0)
+			(type default)
+		)
+	)
+	(wire
+		(pts
 			(xy 54.61 57.15) (xy 54.61 66.04)
 		)
@@
 		)
 	)
-	(wire
-		(pts
-			(xy 152.4 142.24) (xy 152.4 68.58)
-		)
-		(stroke
-			(width 0)
-			(type default)
-		)
-	)
 	(global_label "ST_LINK_SWDIO"
 		(shape input)
@@
 		)
 	)
+	(global_label "ACC_INT1"
+		(shape input)
+		(at 153.67 148.59 270)
+		(fields_autoplaced yes)
+		(effects
+			(font
+				(size 1.27 1.27)
+			)
+			(justify right)
+		)
+		(property "Intersheetrefs" "${INTERSHEET_REFS}"
+			(at 153.67 160.2838 90)
+			(hide yes)
+			(show_name no)
+			(do_not_autoplace no)
+			(effects
+				(font
+					(size 1.27 1.27)
+				)
+				(justify right)
+			)
+		)
+	)
 	(global_label "ST_LINK_GND"
 		(shape input)
@@
 		)
 	)
-	(global_label "I2C_ERR"
-		(shape input)
-		(at 152.4 142.24 270)
-		(fields_autoplaced yes)
-		(effects
-			(font
-				(size 1.27 1.27)
-			)
-			(justify right)
-		)
-		(property "Intersheetrefs" "${INTERSHEET_REFS}"
-			(at 152.4 152.9661 90)
-			(hide yes)
-			(show_name no)
-			(do_not_autoplace no)
-			(effects
-				(font
-					(size 1.27 1.27)
-				)
-				(justify right)
-			)
-		)
-	)
 	(global_label "ST_LINK_RST{slash}RST"
 		(shape input)
@@
 		)
 	)
-	(global_label "LIVE"
-		(shape input)
-		(at 146.05 142.24 270)
-		(effects
-			(font
-				(size 1.27 1.27)
-			)
-			(justify right)
-		)
-		(property "Intersheetrefs" "${INTERSHEET_REFS}"
-			(at 146.05 142.24 90)
-			(hide yes)
-			(show_name no)
-			(do_not_autoplace no)
-			(effects
-				(font
-					(size 1.27 1.27)
-				)
-			)
-		)
-	)
 	(global_label "ST_LIKN_SWCLK"
 		(shape input)
-		(at 247.65 146.05 270)
-		(fields_autoplaced yes)
-		(effects
-			(font
-				(size 1.27 1.27)
-			)
-			(justify right)
-		)
-		(property "Intersheetrefs" "${INTERSHEET_REFS}"
-			(at 247.65 163.6099 90)
-			(hide yes)
-			(show_name no)
+		(at 175.26 147.32 270)
+		(fields_autoplaced yes)
+		(effects
+			(font
+				(size 1.27 1.27)
+			)
+			(justify right)
+		)
+		(property "Intersheetrefs" "${INTERSHEET_REFS}"
+			(at 175.26 164.8799 90)
+			(hide yes)
+			(show_name no)
