File: ghostlight_circuit/programming_connector.kicad_sch (KiCad schematic)
At the start: 1 part, among them J1 Conn_01x08

Commit message: rerouted the board
Connections:
- net V_BAT: now reaches J1.7 (Pin_7)
- net LIVE: no longer names the net of J1.5 (Pin_5)
Changed lines of the file:
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@@
 	(paper "A4")
 	(no_connect
-		(at 107.95 100.33)
+		(at 107.95 95.25)
 	)
 	(wire
@@
 	(wire
 		(pts
-			(xy 80.01 91.44) (xy 101.6 91.44)
-		)
-		(stroke
-			(width 0)
-			(type default)
-		)
-	)
-	(wire
-		(pts
-			(xy 81.28 102.87) (xy 107.95 102.87)
+			(xy 80.01 102.87) (xy 107.95 102.87)
 		)
 		(stroke
@@
 	(wire
 		(pts
-			(xy 81.28 97.79) (xy 107.95 97.79)
-		)
-		(stroke
-			(width 0)
-			(type default)
-		)
-	)
-	(wire
-		(pts
-			(xy 101.6 95.25) (xy 107.95 95.25)
-		)
-		(stroke
-			(width 0)
-			(type default)
-		)
-	)
-	(wire
-		(pts
-			(xy 101.6 91.44) (xy 101.6 95.25)
+			(xy 80.01 95.25) (xy 82.55 95.25)
+		)
+		(stroke
+			(width 0)
+			(type default)
+		)
+	)
+	(wire
+		(pts
+			(xy 81.28 100.33) (xy 107.95 100.33)
+		)
+		(stroke
+			(width 0)
+			(type default)
+		)
+	)
+	(wire
+		(pts
+			(xy 81.28 99.06) (xy 81.28 100.33)
 		)
 		(stroke
@@
 	(wire
 		(pts
+			(xy 82.55 95.25) (xy 82.55 97.79)
+		)
+		(stroke
+			(width 0)
+			(type default)
+		)
+	)
+	(wire
+		(pts
+			(xy 82.55 97.79) (xy 107.95 97.79)
+		)
+		(stroke
+			(width 0)
+			(type default)
+		)
+	)
+	(wire
+		(pts
 			(xy 106.68 87.63) (xy 107.95 87.63)
 		)
@@
 	(wire
 		(pts
+			(xy 80.01 99.06) (xy 81.28 99.06)
+		)
+		(stroke
+			(width 0)
+			(type default)
+		)
+	)
+	(wire
+		(pts
 			(xy 106.68 77.47) (xy 106.68 87.63)
 		)
@@
 		)
 	)
+	(global_label "V_BAT"
+		(shape input)
+		(at 80.01 99.06 180)
+		(fields_autoplaced yes)
+		(effects
+			(font
+				(size 1.27 1.27)
+			)
+			(justify right)
+		)
+		(property "Intersheetrefs" "${INTERSHEET_REFS}"
+			(at 71.6424 99.06 0)
+			(hide yes)
+			(show_name no)
+			(do_not_autoplace no)
+			(effects
+				(font
+					(size 1.27 1.27)
+				)
+				(justify right)
+			)
+		)
+	)
 	(global_label "ST_LINK_VDD"
 		(shape input)
@@
 	(global_label "ST_LINK_GND"
 		(shape input)
-		(at 81.28 102.87 180)
-		(fields_autoplaced yes)
-		(effects
-			(font
-				(size 1.27 1.27)
-			)
-			(justify right)
-		)
-		(property "Intersheetrefs" "${INTERSHEET_REFS}"
-			(at 66.0786 102.87 0)
+		(at 80.01 102.87 180)
+		(fields_autoplaced yes)
+		(effects
+			(font
+				(size 1.27 1.27)
+			)
+			(justify right)
+		)
+		(property "Intersheetrefs" "${INTERSHEET_REFS}"
+			(at 64.8086 102.87 0)
 			(hide yes)
 			(show_name no)
@@
 	(global_label "ST_LINK_RST{slash}RST"
 		(shape input)
-		(at 81.28 97.79 180)
-		(fields_autoplaced yes)
-		(effects
-			(font
-				(size 1.27 1.27)
-			)
-			(justify right)
-		)
-		(property "Intersheetrefs" "${INTERSHEET_REFS}"
-			(at 61.7244 97.79 0)
+		(at 80.01 95.25 180)
+		(fields_autoplaced yes)
+		(effects
+			(font
+				(size 1.27 1.27)
+			)
+			(justify right)
+		)
+		(property "Intersheetrefs" "${INTERSHEET_REFS}"
+			(at 60.4544 95.25 0)
 			(hide yes)
 			(show_name no)
@@
 			)
 		)
-	)
-	(global_label "LIVE"
-		(shape input)
-		(at 80.01 91.44 180)
-		(effects
-			(font
-				(size 1.27 1.27)
-			)
-			(justify right)
-		)
-		(property "Intersheetrefs" "${INTERSHEET_REFS}"
-			(at 80.01 91.44 0)
-			(hide yes)
-			(show_name no)
-			(do_not_autoplace no)
-			(effects
-				(font
-					(size 1.27 1.27)
-				)
-			)
-		)
