File: ghostlight_circuit/led.kicad_sch (KiCad schematic)
At the start: 6 parts, among them IC3 LP5817DRLR

Commit message: update pcb
rerout and connect accelerometer

better re-route
Parts:
- removed BLUE1: TP_B, TestPoint:TestPoint_Pad_D1.0mm, symbol Connector:TestPoint
- removed GREEN1: TP_G, TestPoint:TestPoint_Pad_D1.0mm, symbol Connector:TestPoint
- removed RED1: TP_R, TestPoint:TestPoint_Pad_D1.0mm, symbol Connector:TestPoint
